File: ESP12E Breakout Adapter.brd (EAGLE design)
At the start: 27.5 x 38.8 mm, 16 parts, among them IC1 LM1117MPX-3.3

Commit message: version 1.1
Parts:
- C1: value Tantal 10µF -> 10µF
- C2: value Tantal 22µF -> 22µF
- IC1: value LM1117MPX-3.3 -> LM1117-3.3
Changed lines of the file:
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@@
 <attribute name="VALUE" x="24.00163125" y="36.82948125" size="1.27" layer="27" rot="R270"/>
 </element>
-<element name="IC1" library="lm1117" package="SOT223" value="LM1117MPX-3.3" x="17.67355625" y="32.51655625" smashed="yes" rot="MR0">
+<element name="IC1" library="lm1117" package="SOT223" value="LM1117-3.3" x="17.67355625" y="32.51655625" smashed="yes" rot="MR0">
 <attribute name="NAME" x="20.26435625" y="35.05655625" size="1.27" layer="22" rot="MR90"/>
 </element>
-<element name="C1" library="rcl" package="B/3528-21W" value="Tantal 10µF" x="15.91355625" y="24.56055625" smashed="yes" rot="MR90">
+<element name="C1" library="rcl" package="B/3528-21W" value="10µF" x="15.91355625" y="24.56055625" smashed="yes" rot="MR90">
 <attribute name="NAME" x="17.25955625" y="23.62655625" size="1.27" layer="22" rot="MR90"/>
 </element>
@@
 <element name="JP1" library="pinhead" package="1X02" value="GND | 5V" x="27.180709375" y="11.430640625" smashed="yes" rot="R90"/>
 <element name="JP2" library="pinhead" package="1X02" value="GND | 3V3" x="4.316159375" y="11.426784375" smashed="yes" rot="R270"/>
-<element name="C2" library="rcl" package="B/3528-21W" value="Tantal 22µF" x="11.85955625" y="24.59755625" smashed="yes" rot="MR90">
+<element name="C2" library="rcl" package="B/3528-21W" value="22µF" x="11.85955625" y="24.59755625" smashed="yes" rot="MR90">
 <attribute name="NAME" x="13.20555625" y="23.66355625" size="1.27" layer="22" rot="MR90"/>
 </element>
