File: Breakout Adapter v1.1 - LM1117/ESP12E Breakout Adapter.brd (EAGLE design)
At the start: 27.5 x 38.8 mm, 16 parts, among them IC1 LM1117-3.3

Commit message: kleine änderung
Parts:
- C2: value 22µF -> 10µF
Changed lines of the file:
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@@
 <?xml version="1.0" encoding="utf-8"?>
 <!DOCTYPE eagle SYSTEM "eagle.dtd">
-<eagle version="7.2.2">
+<eagle version="7.3.0">
 <drawing>
 <settings>
@@
 <element name="JP1" library="pinhead" package="1X02" value="GND | 5V" x="27.180709375" y="11.430640625" smashed="yes" rot="R90"/>
 <element name="JP2" library="pinhead" package="1X02" value="GND | 3V3" x="4.316159375" y="11.426784375" smashed="yes" rot="R270"/>
-<element name="C2" library="rcl" package="B/3528-21W" value="22µF" x="11.85955625" y="24.59755625" smashed="yes" rot="MR90">
+<element name="C2" library="rcl" package="B/3528-21W" value="10µF" x="11.85955625" y="24.59755625" smashed="yes" rot="MR90">
 <attribute name="NAME" x="13.20555625" y="23.66355625" size="1.27" layer="22" rot="MR90"/>
 </element>
