File: Breakout Adapter v1.1 - LM1117/ESP12E Breakout Adapter.sch (EAGLE design)
At the start: 16 parts, among them IC1 LM1117-3.3

Commit message: kleine änderung
Parts:
- C2: value 22µF -> 10µF
Changed lines of the file:
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@@
 <?xml version="1.0" encoding="utf-8"?>
 <!DOCTYPE eagle SYSTEM "eagle.dtd">
-<eagle version="7.2.2">
+<eagle version="7.3.0">
 <drawing>
 <settings>
@@
 <part name="JP1" library="pinhead" deviceset="PINHD-1X2" device="" value="GND | 5V"/>
 <part name="JP2" library="pinhead" deviceset="PINHD-1X2" device="" value="GND | 3V3"/>
-<part name="C2" library="rcl" deviceset="CPOL-EU" device="B/3528-21W" value="22µF"/>
+<part name="C2" library="rcl" deviceset="CPOL-EU" device="B/3528-21W" value="10µF"/>
 <part name="R2" library="rcl" deviceset="R-EU_" device="R0805" value="0 Ohm"/>
 <part name="R1" library="rcl" deviceset="R-EU_" device="R0805" value="0 Ohm"/>
