File: Breakout Adapter v2.0D - SPX3819 - Mini/ESP Breakout Adapter - v2_0D - SPX3819 - Mini/ESP Breakout Adapter - v2_0D - SPX3819 - Mini.sch (EAGLE design)
At the start: 26 parts, among them U1 SPX3819

Commit message: mini änderung
Other:
- note added: "LDO Enable"
- moved on the sheet: EN
Changed lines of the file:
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@@
 VCC = 3.3V</text>
 <text x="137.16" y="35.56" size="1.778" layer="91">Led Voltage</text>
+<text x="175.26" y="106.68" size="1.778" layer="91">LDO Enable</text>
 </plain>
 <instances>
@@
 <instance part="C3" gate="G$1" x="109.22" y="129.54"/>
 <instance part="GND7" gate="1" x="66.04" y="109.22"/>
-<instance part="EN" gate="G$1" x="182.88" y="104.14" rot="R270"/>
+<instance part="EN" gate="G$1" x="182.88" y="111.76" rot="R270"/>
 <instance part="R5" gate="G$1" x="218.44" y="134.62" rot="R90"/>
 <instance part="DS" gate="G$1" x="180.34" y="33.02" smashed="yes" rot="R90">
@@
 <attribute name="NAME" x="188.595" y="133.35" size="1.778" layer="95"/>
 </instance>
-<instance part="VIN" gate="G$1" x="50.8" y="121.92" rot="R270"/>
+<instance part="VIN" gate="G$1" x="50.8" y="121.92" smashed="yes" rot="R270">
+<attribute name="NAME" x="52.07" y="118.745" size="1.778" layer="95" rot="R180"/>
+</instance>
 <instance part="LED_VOLTAGE" gate="G$1" x="144.78" y="22.86" smashed="yes" rot="R90">
 <attribute name="VALUE" x="146.685" y="25.4" size="1.778" layer="96" rot="R90"/>
@@
 </segment>
 <segment>
-<wire x1="182.88" y1="106.68" x2="182.88" y2="114.3" width="0.1524" layer="91"/>
+<wire x1="182.88" y1="114.3" x2="182.88" y2="124.46" width="0.1524" layer="91"/>
 <pinref part="EN" gate="G$1" pin="1"/>
-<junction x="182.88" y="114.3"/>
-<label x="182.88" y="116.84" size="1.778" layer="95"/>
-</segment>
-</net>
+<junction x="182.88" y="124.46"/>
+<label x="182.88" y="124.46" size="1.778" layer="95"/>
+</segment>
+</net>
