File: Breakout Adapter v3.0A - AS1363 - Mini/ESP Breakout Adapter - v3_0A - AS1363 - Mini/ESP Breakout Adapter - v3_0A - AS1363 - Mini.brd (EAGLE design)
At the start: 24.3 x 30.6 mm, 27 parts

Commit message: neue versionierung
Other:
- board text added: "3.0A"
- board text added: "ESP8266 Breakout AS Mini Adapter v3.0A VIN=3.5-5.5V (500mA) Iq=40µA, Ishdn=<1µA"
- board text removed: "2.0C"
- board text removed: "ESP8266 Breakout AS Mini Adapter v2.0C VIN=3.5-5.5V (500mA) Iq=40µA, Ishdn=<1µA"
Changed lines of the file:
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@@
 <text x="23.495" y="23.114" size="0.8128" layer="21" ratio="12" rot="R270">Rx</text>
 <text x="23.495" y="25.654" size="0.8128" layer="21" ratio="12" rot="R270">Tx</text>
-<text x="4.2799" y="25.1333" size="0.6096" layer="21" ratio="12" rot="R90">2.0C</text>
+<text x="4.2799" y="25.1333" size="0.6096" layer="21" ratio="12" rot="R90">3.0A</text>
 <text x="9.54040625" y="8.916303125" size="0.8128" layer="21">Okt, 2015</text>
 <text x="23.47268125" y="2.835553125" size="0.8128" layer="21" ratio="12" rot="R270">EN</text>
@@
 <text x="9.9187" y="1.4605" size="0.8128" layer="21" ratio="12" rot="R180">Reset</text>
 <text x="12.319" y="29.6545" size="0.8128" layer="22" ratio="12" rot="MR0" align="top-center">ESP8266 Breakout
-AS Mini Adapter v2.0C
+AS Mini Adapter v3.0A
 VIN=3.5-5.5V (500mA)
 Iq=40µA, Ishdn=&lt;1µA</text>
@@
 <wire x1="22.606" y1="10.922" x2="21.336" y2="12.192" width="0.127" layer="21" curve="-90"/>
 <wire x1="21.336" y1="12.192" x2="22.733" y2="13.462" width="0.127" layer="21" curve="-90"/>
-<text x="20.4851" y="27.3177" size="0.6096" layer="21" ratio="12" rot="R270">2.0C</text>
+<text x="20.4851" y="27.3177" size="0.6096" layer="21" ratio="12" rot="R270">3.0A</text>
 <text x="12.446" y="23.0505" size="0.8128" layer="21" ratio="12" align="top-center">ESP8266 Breakout
 AS Mini Adapter</text>
