File: Breakout Adapter v3.0B - SPX3819 - Mini/ESP Breakout Adapter - v3_0B - SPX3819 - Mini/ESP Breakout Adapter - v3_0B - SPX3819 - Mini.brd (EAGLE design)
At the start: 24.3 x 30.6 mm, 27 parts, among them U1 SPX3819

Commit message: neue versionierung
Other:
- board text added: "3.0B"
- board text added: "ESP8266 Breakout SPX Mini Adapter v3.0B VIN=3.8-16V (500mA) Iq=90µA, Ishdn=<1µA"
- board text removed: "2.0D"
- board text removed: "ESP8266 Breakout SPX Mini Adapter v2.0D VIN=3.8-16V (500mA) Iq=90µA, Ishdn=<1µA"
Changed lines of the file:
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@@
 <text x="9.9187" y="1.4605" size="0.8128" layer="21" ratio="12" rot="R180">Reset</text>
 <text x="12.319" y="29.6545" size="0.8128" layer="22" ratio="12" rot="MR0" align="top-center">ESP8266 Breakout
-SPX Mini Adapter v2.0D
+SPX Mini Adapter v3.0B
 VIN=3.8-16V (500mA)
 Iq=90µA, Ishdn=&lt;1µA</text>
@@
 <text x="5.08" y="5.842" size="0.6096" layer="21" ratio="12">hold down Flash during Reset</text>
 <text x="9.906" y="6.985" size="0.6096" layer="21" ratio="12">UART boot: </text>
-<text x="20.4851" y="27.3177" size="0.6096" layer="21" ratio="12" rot="R270">2.0D</text>
+<text x="20.4851" y="27.3177" size="0.6096" layer="21" ratio="12" rot="R270">3.0B</text>
 <text x="12.446" y="23.0505" size="0.8128" layer="21" ratio="12" align="top-center">ESP8266 Breakout
 SPX Mini Adapter</text>
-<text x="4.2799" y="25.1333" size="0.6096" layer="21" ratio="12" rot="R90">2.0D</text>
+<text x="4.2799" y="25.1333" size="0.6096" layer="21" ratio="12" rot="R90">3.0B</text>
 </plain>
 <attributes>
