File: Breakout Adapter v3.0B - SPX3819 - Mini/ESP Breakout Adapter - v3_0B - SPX3819 - Mini/ESP Breakout Adapter - v3_0B - SPX3819 - Mini.sch (EAGLE design)
At the start: 26 parts, among them U1 SPX3819

Commit message: neue versionierung
Other:
- note added: "ESP8266 Breakout - ESP-07/ESP-12 SPX Mini Adapter v3.0B Date: 17. Oktober 2015 License: CC-BY-SA By: Johannes S. (joh.raspi) github.com/8n1/ESP8266-Breakout-Adapter"
- note removed: "ESP8266 Breakout - ESP-07/ESP-12 SPX Mini Adapter v2.0D Date: 17. Oktober 2015 License: CC-BY-SA By: Johannes S. (joh.raspi) github.com/8n1/ESP8266-Breakout-Adapter"
Changed lines of the file:
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@@
 <plain>
 <text x="165.1" y="-10.16" size="1.778" layer="91">ESP8266 Breakout - ESP-07/ESP-12
-SPX Mini Adapter v2.0D
+SPX Mini Adapter v3.0B
 Date: 17. Oktober 2015
 License: CC-BY-SA
